File: pcb/duckiebot_pwm_shield.brd (EAGLE design)
At the start: 66 x 57 mm, 13 parts, among them J1 RASPBERRYPI-40-PIN-GPIO

Commit message: v1.3, falta arreglar el layer del pato ql
Parts:
- added U$1: (no value), uchile_robotics_eagle_lib:DUCK_LOGO
- renumbered J2 to H-BRIDGE, J3 to PWR
Other:
- board text added: "Duckiebot Shield V1.3"
- board text removed: "Duckiebot Shield V1.0"
Changed lines of the file:
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@@
 <hole x="62" y="3" drill="3.2"/>
 <hole x="62" y="52" drill="3.2"/>
-<wire x1="38.2" y1="30" x2="38.2" y2="1" width="0.254" layer="51"/>
+<wire x1="38.2" y1="30" x2="38.2" y2="1" width="0.254" layer="25"/>
 <wire x1="38.2" y1="1" x2="63.2" y2="1" width="0.254" layer="51"/>
 <wire x1="63.2" y1="1" x2="63.2" y2="30" width="0.254" layer="51"/>
-<wire x1="63.2" y1="30" x2="38.2" y2="30" width="0.254" layer="51"/>
-<text x="23.2" y="35" size="2.54" layer="1" font="vector" ratio="18">Duckiebot
+<wire x1="63.2" y1="30" x2="38.2" y2="30" width="0.254" layer="25"/>
+<text x="23.2" y="35" size="2.54" layer="25" font="vector" ratio="18">Duckiebot
 Shield
-V1.0</text>
-<text x="32.4" y="2.8" size="2.54" layer="1" font="vector" ratio="14">+</text>
-<text x="8" y="8" size="2.54" layer="1" font="vector" ratio="14">-</text>
+V1.3</text>
+<text x="32.4" y="3.2" size="2.54" layer="25" font="vector" ratio="14">+</text>
+<text x="7.2" y="7" size="2.54" layer="25" font="vector" ratio="14">-</text>
 </plain>
 <attributes>
@@
 <elements>
 <element name="J1" library="SparkFun-Boards" package="2X20-SHROUDED" value="RASPBERRYPI-40-PIN-GPIO" x="33" y="52" rot="R90"/>
-<element name="J2" library="SparkFun-Connectors" package="1X06_LONGPADS" value="" x="57.2" y="26.4" rot="R180"/>
+<element name="H-BRIDGE" library="SparkFun-Connectors" package="1X06_LONGPADS" value="" x="57.2" y="26.4" rot="R180"/>
 <element name="U$2" library="Arduino-clone" package="PRO-MINI" value="PRO-MINI" x="10.78" y="14.76"/>
-<element name="J3" library="con-jack" package="SPC4077" value="" x="55.6" y="37.4" rot="R180">
+<element name="PWR" library="con-jack" package="SPC4077" value="" x="55.6" y="37.4" smashed="yes" rot="R180">
 <attribute name="MF" value="" x="55.6" y="37.4" size="1.778" layer="27" rot="R180" display="off"/>
 <attribute name="MPN" value="" x="55.6" y="37.4" size="1.778" layer="27" rot="R180" display="off"/>
 <attribute name="OC_NEWARK" value="unknown" x="55.6" y="37.4" size="1.778" layer="27" rot="R180" display="off"/>
 <attribute name="OC_FARNELL" value="unknown" x="55.6" y="37.4" size="1.778" layer="27" rot="R180" display="off"/>
-</element>
-<element name="SERVO1" library="SparkFun-Connectors" package="1X03_LONGPADS" value="" x="12" y="3" rot="R90"/>
-<element name="SERVO2" library="SparkFun-Connectors" package="1X03_LONGPADS" value="" x="18.6" y="3" rot="R90"/>
+<attribute name="NAME" x="57.56" y="32.52" size="1.27" layer="25" rot="R180"/>
+<attribute name="VALUE" x="65.76" y="43.75" size="1.27" layer="27" rot="R180"/>
+</element>
+<element name="SERVO1" library="SparkFun-Connectors" package="1X03_LONGPADS" value="" x="12" y="3" smashed="yes" rot="R90">
+<attribute name="NAME" x="9.5362" y="1.6538" size="1.016" layer="25" ratio="10" rot="R90"/>
+<attribute name="VALUE" x="15.81" y="1.73" size="1.27" layer="27" rot="R90"/>
+</element>
+<element name="SERVO2" library="SparkFun-Connectors" package="1X03_LONGPADS" value="" x="18.6" y="3" smashed="yes" rot="R90">
+<attribute name="NAME" x="16.1362" y="1.6538" size="1.016" layer="25" ratio="10" rot="R90"/>
+<attribute name="VALUE" x="22.41" y="1.73" size="1.27" layer="27" rot="R90"/>
+</element>
 <element name="IMU" library="SparkFun-Connectors" package="1X04_LONGPADS" value="" x="25.6" y="7.8">
 <attribute name="PROD_ID" value="CONN-09696" x="25.6" y="7.8" size="1.778" layer="27" display="off"/>
 </element>
-<element name="SONAR1" library="SparkFun-Connectors" package="1X04_LONGPADS" value="" x="33.2" y="19.6" rot="R180">
+<element name="SONAR1" library="SparkFun-Connectors" package="1X04_LONGPADS" value="" x="33.2" y="19.6" smashed="yes" rot="R180">
 <attribute name="PROD_ID" value="CONN-09696" x="33.2" y="19.6" size="1.778" layer="27" rot="R180" display="off"/>
-</element>
-<element name="SONAR2" library="SparkFun-Connectors" package="1X04_LONGPADS" value="" x="33.2" y="15" rot="R180">
+<attribute name="NAME" x="34.8638" y="22.3462" size="0.8128" layer="25" ratio="10" rot="R270"/>
+<attribute name="VALUE" x="34.47" y="23.41" size="1.27" layer="27" rot="R180"/>
+</element>
+<element name="SONAR2" library="SparkFun-Connectors" package="1X04_LONGPADS" value="" x="33.2" y="15" smashed="yes" rot="R180">
 <attribute name="PROD_ID" value="CONN-09696" x="33.2" y="15" size="1.778" layer="27" rot="R180" display="off"/>
-</element>
-<element name="ENC1" library="SparkFun-Connectors" package="1X03_LONGPADS" value="" x="30.8" y="31.2" rot="R180"/>
-<element name="ENC2" library="SparkFun-Connectors" package="1X03_LONGPADS" value="" x="30.8" y="26.6" rot="R180"/>
-<element name="R1" library="adafruit" package="0204/5" value="1k" x="11.8" y="36.2" rot="R180"/>
-<element name="R2" library="adafruit" package="0204/5" value="1k" x="11.8" y="39.6" rot="R180"/>
+<attribute name="NAME" x="34.8638" y="16.9462" size="0.8128" layer="25" ratio="10" rot="R270"/>
+<attribute name="VALUE" x="34.47" y="18.81" size="1.27" layer="27" rot="R180"/>
+</element>
+<element name="ENC1" library="SparkFun-Connectors" package="1X03_LONGPADS" value="" x="30.8" y="31.2" smashed="yes" rot="R180">
+<attribute name="NAME" x="24.1362" y="29.2538" size="1.016" layer="25" ratio="10" rot="R90"/>
+<attribute name="VALUE" x="32.07" y="35.01" size="1.27" layer="27" rot="R180"/>
+</element>
+<element name="ENC2" library="SparkFun-Connectors" package="1X03_LONGPADS" value="" x="30.8" y="26.6" smashed="yes" rot="R180">
+<attribute name="NAME" x="23.2638" y="28.5462" size="1.016" layer="25" ratio="10" rot="R270"/>
+<attribute name="VALUE" x="32.07" y="30.41" size="1.27" layer="27" rot="R180"/>
+</element>
+<element name="R1" library="adafruit" package="0204/5" value="1k" x="11.8" y="36.2" smashed="yes" rot="R180">
+<attribute name="NAME" x="10.4066" y="35.0316" size="0.9906" layer="25" ratio="12" rot="R180"/>
+<attribute name="VALUE" x="12.1336" y="34.9114" size="0.9906" layer="27" ratio="12" rot="R180"/>
+</element>
+<element name="R2" library="adafruit" package="0204/5" value="1k" x="11.8" y="39.6" smashed="yes" rot="R180">
+<attribute name="NAME" x="10.0066" y="41.8316" size="0.9906" layer="25" ratio="12" rot="R180"/>
+<attribute name="VALUE" x="12.1336" y="41.7114" size="0.9906" layer="27" ratio="12" rot="R180"/>
+</element>
+<element name="U$1" library="uchile_robotics_eagle_lib" package="DUCK_LOGO" value="" x="36" y="31.6"/>
 </elements>
 <signals>
@@
 <contactref element="J1" pad="34"/>
 <contactref element="J1" pad="39"/>
-<contactref element="J3" pad="1"/>
-<contactref element="J3" pad="2"/>
+<contactref element="PWR" pad="1"/>
+<contactref element="PWR" pad="2"/>
 <contactref element="U$2" pad="GND"/>
 <contactref element="J1" pad="9"/>
-<contactref element="J2" pad="4"/>
+<contactref element="H-BRIDGE" pad="4"/>
 <wire x1="58.6" y1="37.4" x2="58.6" y2="40.4" width="0.4064" layer="16"/>
 <wire x1="58.6" y1="40.4" x2="55.6" y2="42.2" width="0.4064" layer="16"/>
@@
 </signal>
 <signal name="VCC">
-<contactref element="J3" pad="3"/>
-<contactref element="J2" pad="3"/>
+<contactref element="PWR" pad="3"/>
+<contactref element="H-BRIDGE" pad="3"/>
 <contactref element="SERVO1" pad="2"/>
 <contactref element="SERVO2" pad="2"/>
@@
 <signal name="B-1A">
 <contactref element="U$2" pad="D12"/>
-<contactref element="J2" pad="6"/>
+<contactref element="H-BRIDGE" pad="6"/>
 <wire x1="22.8" y1="23.8" x2="21.4" y2="22.4" width="0.4064" layer="1"/>
 <wire x1="21.4" y1="22.4" x2="14.8" y2="22.4" width="0.4064" layer="1"/>
@@
 <signal name="B-1B">
 <contactref element="U$2" pad="D6"/>
-<contactref element="J2" pad="5"/>
+<contactref element="H-BRIDGE" pad="5"/>
 <wire x1="4.43" y1="21.11" x2="6.89" y2="21.11" width="0.4064" layer="16"/>
 <wire x1="6.89" y1="21.11" x2="7.8" y2="20.2" width="0.4064" layer="16"/>
@@
 <signal name="A-1B">
 <contactref element="U$2" pad="D5"/>
-<contactref element="J2" pad="1"/>
+<contactref element="H-BRIDGE" pad="1"/>
 <wire x1="57.2" y1="26.4" x2="57.2" y2="20" width="0.4064" layer="16"/>
 <wire x1="57.2" y1="20" x2="47.6" y2="10.4" width="0.4064" layer="16"/>
@@
 <signal name="A-1A">
 <contactref element="U$2" pad="D11"/>
-<contactref element="J2" pad="2"/>
+<contactref element="H-BRIDGE" pad="2"/>
 <wire x1="54.66" y1="26.4" x2="54.66" y2="20.66" width="0.4064" layer="16"/>
 <wire x1="54.66" y1="20.66" x2="45.8" y2="11.8" width="0.4064" layer="16"/>

Commit message: fixed resistor size, v1.4 ready to build
Parts:
- R1, R2: device adafruit:0204/5 -> resistor:0309/10
- moved R1 1.08 mm to (12.2, 35.2)
- moved R2 0.57 mm to (12.2, 40.0)
Routing:
- net N$3: track 50.3 -> 39.8 mm, vias 0 -> 1
- net N$4: track 31.5 -> 34.8 mm
- net N$2: track 5.59 -> 4.12 mm
Other:
- board text added: "Duckiebot Shield V1.4"
- board text removed: "Duckiebot Shield V1.3"
Changed lines of the file:
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@@
 <?xml version="1.0" encoding="utf-8"?>
 <!DOCTYPE eagle SYSTEM "eagle.dtd">
-<eagle version="7.7.0">
+<eagle version="7.6.0">
 <drawing>
 <settings>
@@
 <text x="23.2" y="35" size="2.54" layer="25" font="vector" ratio="18">Duckiebot
 Shield
-V1.3</text>
+V1.4</text>
 <text x="32.4" y="3.2" size="2.54" layer="25" font="vector" ratio="14">+</text>
 <text x="7.2" y="7" size="2.54" layer="25" font="vector" ratio="14">-</text>
@@
 <attribute name="VALUE" x="32.07" y="30.41" size="1.27" layer="27" rot="R180"/>
 </element>
-<element name="R1" library="adafruit" package="0204/5" value="1k" x="11.8" y="36.2" smashed="yes" rot="R180">
-<attribute name="NAME" x="10.4066" y="35.0316" size="0.9906" layer="25" ratio="12" rot="R180"/>
-<attribute name="VALUE" x="12.1336" y="34.9114" size="0.9906" layer="27" ratio="12" rot="R180"/>
-</element>
-<element name="R2" library="adafruit" package="0204/5" value="1k" x="11.8" y="39.6" smashed="yes" rot="R180">
-<attribute name="NAME" x="10.0066" y="41.8316" size="0.9906" layer="25" ratio="12" rot="R180"/>
-<attribute name="VALUE" x="12.1336" y="41.7114" size="0.9906" layer="27" ratio="12" rot="R180"/>
+<element name="R1" library="resistor" package="0309/10" value="1k" x="12.2" y="35.2" smashed="yes" rot="R180">
+<attribute name="NAME" x="10.8066" y="35.6316" size="0.9906" layer="25" ratio="12" rot="R180"/>
+<attribute name="VALUE" x="14.7336" y="35.7114" size="0.9906" layer="27" ratio="12" rot="R180"/>
+</element>
+<element name="R2" library="resistor" package="0309/10" value="1k" x="12.2" y="40" smashed="yes" rot="R180">
+<attribute name="NAME" x="10.8066" y="40.4316" size="0.9906" layer="25" ratio="12" rot="R180"/>
+<attribute name="VALUE" x="14.5336" y="40.5114" size="0.9906" layer="27" ratio="12" rot="R180"/>
 </element>
 <element name="U$1" library="uchile_robotics_eagle_lib" package="DUCK_LOGO" value="" x="36" y="31.6"/>
@@
 <contactref element="U$2" pad="RX1"/>
 <contactref element="R1" pad="2"/>
-<wire x1="4.43" y1="38.89" x2="6.57" y2="38.89" width="0.4064" layer="16"/>
-<wire x1="6.57" y1="38.89" x2="9.26" y2="36.2" width="0.4064" layer="16"/>
+<wire x1="4.43" y1="38.89" x2="5.71" y2="38.89" width="0.4064" layer="16"/>
+<wire x1="5.71" y1="38.89" x2="7.2" y2="37.4" width="0.4064" layer="16"/>
+<wire x1="7.2" y1="37.4" x2="7.2" y2="35.28" width="0.4064" layer="16"/>
+<wire x1="7.2" y1="35.28" x2="7.12" y2="35.2" width="0.4064" layer="16"/>
 </signal>
 <signal name="RAW">
@@
 <contactref element="U$2" pad="TX0"/>
 <contactref element="R2" pad="2"/>
-<wire x1="4.43" y1="41.43" x2="7.43" y2="41.43" width="0.4064" layer="16"/>
-<wire x1="7.43" y1="41.43" x2="9.26" y2="39.6" width="0.4064" layer="16"/>
+<wire x1="4.43" y1="41.43" x2="7.12" y2="41.43" width="0.4064" layer="16"/>
+<wire x1="7.12" y1="41.43" x2="7.12" y2="40" width="0.4064" layer="16"/>
 </signal>
 <signal name="VCC">
@@
 <contactref element="J1" pad="10"/>
 <contactref element="R2" pad="1"/>
-<wire x1="14.34" y1="39.6" x2="16.2" y2="37.74" width="0.4064" layer="1"/>
-<wire x1="16.2" y1="37.74" x2="16.2" y2="35.2" width="0.4064" layer="1"/>
-<wire x1="16.2" y1="35.2" x2="15.4" y2="34.4" width="0.4064" layer="1"/>
-<wire x1="15.4" y1="34.4" x2="7.2" y2="34.4" width="0.4064" layer="1"/>
-<wire x1="7.2" y1="34.4" x2="7" y2="34.6" width="0.4064" layer="1"/>
-<wire x1="7" y1="34.6" x2="7" y2="46.2" width="0.4064" layer="1"/>
-<wire x1="7" y1="46.2" x2="5.8" y2="47.4" width="0.4064" layer="1"/>
-<wire x1="5.8" y1="47.4" x2="5.8" y2="54.8" width="0.4064" layer="1"/>
-<wire x1="5.8" y1="54.8" x2="6.8" y2="55.8" width="0.4064" layer="1"/>
-<wire x1="6.8" y1="55.8" x2="16.8" y2="55.8" width="0.4064" layer="1"/>
-<wire x1="16.8" y1="55.8" x2="19.03" y2="53.57" width="0.4064" layer="1"/>
-<wire x1="19.03" y1="53.57" x2="19.03" y2="53.27" width="0.4064" layer="1"/>
+<wire x1="17.28" y1="40" x2="15.88" y2="41.4" width="0.4064" layer="16"/>
+<wire x1="15.88" y1="41.4" x2="12.2" y2="41.4" width="0.4064" layer="16"/>
+<wire x1="12.2" y1="41.4" x2="12" y2="41.6" width="0.4064" layer="16"/>
+<wire x1="12" y1="41.6" x2="12" y2="46.4" width="0.4064" layer="16"/>
+<wire x1="12" y1="46.4" x2="11.2" y2="47.2" width="0.4064" layer="16"/>
+<wire x1="11.2" y1="47.2" x2="5.4" y2="47.2" width="0.4064" layer="16"/>
+<via x="5.4" y="47.2" extent="1-16" drill="0.6" shape="octagon"/>
+<wire x1="5.4" y1="47.2" x2="5.4" y2="53.8" width="0.4064" layer="1"/>
+<wire x1="5.4" y1="53.8" x2="7.4" y2="55.8" width="0.4064" layer="1"/>
+<wire x1="7.4" y1="55.8" x2="16.5" y2="55.8" width="0.4064" layer="1"/>
+<wire x1="16.5" y1="55.8" x2="19.03" y2="53.27" width="0.4064" layer="1"/>
 </signal>
 <signal name="N$4">
 <contactref element="R1" pad="1"/>
 <contactref element="J1" pad="8"/>
-<wire x1="16.49" y1="53.27" x2="14.76" y2="55" width="0.4064" layer="1"/>
-<wire x1="14.76" y1="55" x2="7.6" y2="55" width="0.4064" layer="1"/>
-<wire x1="7.6" y1="55" x2="7.2" y2="54.6" width="0.4064" layer="1"/>
-<wire x1="7.2" y1="54.6" x2="7.2" y2="48" width="0.4064" layer="1"/>
-<wire x1="7.2" y1="48" x2="9.6" y2="45.6" width="0.4064" layer="1"/>
-<wire x1="9.6" y1="45.6" x2="9.6" y2="41.6" width="0.4064" layer="1"/>
-<wire x1="9.6" y1="41.6" x2="14.34" y2="36.86" width="0.4064" layer="1"/>
-<wire x1="14.34" y1="36.86" x2="14.34" y2="36.2" width="0.4064" layer="1"/>
+<wire x1="16.49" y1="53.27" x2="14.96" y2="54.8" width="0.4064" layer="1"/>
+<wire x1="14.96" y1="54.8" x2="8" y2="54.8" width="0.4064" layer="1"/>
+<wire x1="8" y1="54.8" x2="7.2" y2="54" width="0.4064" layer="1"/>
+<wire x1="7.2" y1="54" x2="7.2" y2="49.4" width="0.4064" layer="1"/>
+<wire x1="7.2" y1="49.4" x2="9.4" y2="47.2" width="0.4064" layer="1"/>
+<wire x1="9.4" y1="47.2" x2="9.4" y2="40.4" width="0.4064" layer="1"/>
+<wire x1="9.4" y1="40.4" x2="14.6" y2="35.2" width="0.4064" layer="1"/>
+<wire x1="14.6" y1="35.2" x2="17.28" y2="35.2" width="0.4064" layer="1"/>
 </signal>
 <signal name="D13">
